File: LOW_LEVEL/Roblip6_lowlevel_eagles_files/robLip6_lowlevel.sch (EAGLE design)
At the start: 3 parts, among them X1 741256-49

Commit message: commit pcb
Parts:
- removed X1: 741256-49, con-conrad:741256-49
- added JP1: (no value), pinhead:PINHD-1X8
- added JP11: (no value), pinhead:PINHD-1X6
- added ROUES_DROITES, ROUES_GAUCHES, SERVO0, SERVO1, SERVO2, SERVO3, SERVO4, SERVO5, TOURELLE: (no value), pinhead:PINHD-1X3/90
Connections:
- removed net GND@2: U$1G$3.GND@2, X1-2.KL
- removed net N$1: R1.2, U$1G$2.50
- removed net N$2: U$1G$2.40, X1-3.KL
- removed net N$3: U$1G$2.34, X1-4.KL
- removed net N$4: U$1G$2.41
- new net +3V3: U$1G$1.AREF, U$1G$2.+V, U$1G$3.+V
- new net +5V: JP1.1, JP11.1, R1.1, ROUES_DROITES.2, ROUES_GAUCHES.2, SERVO0.2, SERVO1.2, SERVO2.2, SERVO3.2, SERVO4.2, SERVO5.2, TOURELLE.2, U$1G$2.RAW
- new net GND: JP1.2, JP11.6, ROUES_DROITES.1, ROUES_GAUCHES.1, SERVO0.1, SERVO1.1, SERVO2.1, SERVO3.1, SERVO4.1, SERVO5.1, TOURELLE.1, U$1G$1.GND, U$1G$2.GND@2, U$1G$3.GND@1, U$1G$3.GND@2, U$1G$3.GND@3
- new net GND@1: U$1G$2.GND@1
- new net IMU_RX: JP1.4, U$1G$2.34
- new net IMU_TX: JP1.3, U$1G$2.40
- new net RD: ROUES_DROITES.3, U$1G$3.79
- new net RG: ROUES_GAUCHES.3, U$1G$3.78
- new net S0: SERVO0.3, U$1G$3.57
- new net S1: SERVO1.3, U$1G$3.58
- new net S2: SERVO2.3, U$1G$3.66
- new net S3: SERVO3.3, U$1G$3.67
- new net S4: SERVO4.3, U$1G$3.74
- new net S5: SERVO5.3, U$1G$3.75
- new net SCL_LIDAR: JP11.4, U$1G$2.51
- new net SDA_LIDAR: JP11.5, R1.2, U$1G$2.50
- new net ST: TOURELLE.3, U$1G$3.80
- net RAW: now also U$1G$3.RAW; no longer R1.1, U$1G$2.RAW, X1-1.KL
Other:
- note added: "ACTIONNEURS"
- note added: "ADC"
- note added: "CAPTEURS"
- note added: "IMU"
- note added: "LIDAR"
- note added: "ROUES_DROITE"
- note added: "ROUES_GAUCHE"
- note added: "SERVO_0"
- note added: "SERVO_1"
- note added: "SERVO_2"
- note added: "SERVO_3"
- note added: "SERVO_4"
- note added: "SERVO_5"
- note added: "SERVO_TOURELLE"
- moved on the sheet: R1
